File: lab4/KiCad/Lab4.kicad_pcb (KiCad board)
At the start: 2 copper layers, 120 x 234 mm, 287 parts, among them J1 Sense test points, J10 CAN A isolation, J11 CAN A test, J14 CAN B isolation, J15 CAN B test, J2 Current test, J20 CAN A isolation, J21 CAN A test, J24 CAN B isolation, J25 CAN B test, J3 Current test, J30 CAN A isolation, J31 CAN A test, J34 CAN B isolation, J35 CAN B test, J40 Battery input: 1=+ 2=GND, J41 VBAT test, J42 Rail / PG / GND, J43 Rail / PG / GND, J44 Rail / PG / GND, J500 BOOT recovery, J501 SWD (2.54mm), J502 3.3V TTL UART, J503 LAB3 rows 1-13, J504 Additional probes, J505 Reserved / encoder probes, J550 FRONT LEFT lamp, J551 FRONT RIGHT lamp, J600 BOOT recovery, J601 SWD (2.54mm), J602 3.3V TTL UART, J603 LAB3 rows 1-13, J604 Additional probes, J605 Reserved / encoder probes, J650 REAR LEFT lamp, J651 REAR RIGHT lamp, J70 Raspberry Pi4 GPIO, J703 LAB3 rows 1-13, J704 Pi extra probes, J80 LEFT motor, J81 RIGHT motor, J82 LEFT encoder, J83 RIGHT encoder, J90 Servo: GND / 6.6V / PWM, Q1 DMPH3010LK3-13, Q550 MMBT3904, Q551 MMBT3904, Q650 MMBT3904, Q651 MMBT3904, U1 INA180A2IDBVR, U10 MCP2515T-I/ST, U11 SN65HVD231DR, U14 MCP2515T-I/ST, U15 SN65HVD231DR, U2 ACS712ELCTR-05B-T, U20 MCP2515T-I/ST, U21 SN65HVD231DR, U24 MCP2515T-I/ST, U25 SN65HVD231DR, U3 ACS712ELCTR-05B-T, U30 MCP2515T-I/ST, U31 SN65HVD231DR, U34 MCP2515T-I/ST, U35 SN65HVD231DR, U40 TPS564252DRLR, U41 TPS564252DRLR, U42 TPS564252DRLR, U50 STM32F401RET6TR, U60 STM32F401RET6TR, U80 L298N, U81 SN74LVC14APWR, Y10 16 MHz, Y14 16 MHz, Y20 16 MHz, Y24 16 MHz, Y30 16 MHz, Y34 16 MHz

Commit message: Prepare Lab 4 review package and align course assembly plan
Parts:
- R1: footprint Resistor_SMD:R_2512_6332Metric -> Lab4_Power:Vishay_WSL2512_7m_to_500m
Other:
- board text added: "6396BG 41.91x25.4 ENVELOPE / MOUNT TO VERIFY"
- board text removed: "L298 HEATSINK ENVELOPE TO VERIFY"

Commit message: Reconcile Lab 4 review schematic, sourcing and verification
Parts:
- H5, H6, H7, H8: value Pi support <=5mm hardware OD -> Pi support <=5.5mm hardware OD; footprint Lab4_Mechanical:Pi_support_M2.5_D5.0 -> Lab4_Mechanical:Pi_support_M2.5_D5.5
Connections:
- J82 pad 1: /+5V -> /+3V3
- J83 pad 1: /+5V -> /+3V3
