File: lab4/KiCad/Front.kicad_sch (KiCad schematic)
At the start: 34 parts, among them J1 Sense test points, J10 CAN A isolation, J11 CAN A test, J14 CAN B isolation, J15 CAN B test, U1 INA180A2IDBVR, U10 MCP2515T-I/ST, U11 SN65HVD231MDREP, U14 MCP2515T-I/ST, U15 SN65HVD231MDREP, Y10 16 MHz, Y14 16 MHz

Commit message: Integrate Lab 4 MCU support, diagnostics and hierarchical connections
Parts:
- added C500: 100n VDD19, Capacitor_SMD:C_0603_1608Metric, symbol Device:C
- added C501: 100n VDD32, Capacitor_SMD:C_0603_1608Metric, symbol Device:C
- added C502: 100n VDD48, Capacitor_SMD:C_0603_1608Metric, symbol Device:C
- added C503: 100n VDD64, Capacitor_SMD:C_0603_1608Metric, symbol Device:C
- added C504: 100n VBAT, Capacitor_SMD:C_0603_1608Metric, symbol Device:C
- added C505: 4.7u VDD bulk, Capacitor_SMD:C_0805_2012Metric, symbol Device:C
- added C506: 4.7u VCAP1, Capacitor_SMD:C_0805_2012Metric, symbol Device:C
- added C507: 100n VDDA, Capacitor_SMD:C_0603_1608Metric, symbol Device:C
- added C508: 1u VDDA, Capacitor_SMD:C_0603_1608Metric, symbol Device:C
- added C509: 100n NRST, Capacitor_SMD:C_0603_1608Metric, symbol Device:C
- added C510: 100n TEST, Capacitor_SMD:C_0603_1608Metric, symbol Device:C
- added D510: STATUS green, LED_SMD:LED_0603_1608Metric, symbol Device:LED
- added D511: ERR red, LED_SMD:LED_0603_1608Metric, symbol Device:LED
- added D512: DEG_A yellow, LED_SMD:LED_0603_1608Metric, symbol Device:LED
- added D513: DEG_B yellow, LED_SMD:LED_0603_1608Metric, symbol Device:LED
- added FB50: 600R @100MHz, Inductor_SMD:L_0603_1608Metric, symbol Device:FerriteBead
- added J500: BOOT recovery, Connector_PinHeader_2.54mm:PinHeader_1x02_P2.54mm_Vertical, symbol Connector_Generic:Conn_01x02
- added J501: SWD (2.54mm), Connector_PinHeader_2.54mm:PinHeader_1x06_P2.54mm_Vertical, symbol Connector_Generic:Conn_01x06
- added J502: 3.3V TTL UART, Connector_PinHeader_2.54mm:PinHeader_1x03_P2.54mm_Vertical, symbol Connector_Generic:Conn_01x03
- added J503: LAB3 rows 1-13, Connector_PinHeader_2.54mm:PinHeader_1x13_P2.54mm_Vertical, symbol Connector_Generic:Conn_01x13
- added J504: Additional probes, Connector_PinHeader_2.54mm:PinHeader_1x08_P2.54mm_Vertical, symbol Connector_Generic:Conn_01x08
- added J505: Reserved / encoder probes, Connector_PinHeader_2.54mm:PinHeader_1x04_P2.54mm_Vertical, symbol Connector_Generic:Conn_01x04
- added R500: 10k BOOT0, Resistor_SMD:R_0603_1608Metric, symbol Device:R
- added R501: 10k NRST, Resistor_SMD:R_0603_1608Metric, symbol Device:R
- added R502: 10k TEST pullup, Resistor_SMD:R_0603_1608Metric, symbol Device:R
- added R510, R511, R512, R513: 1k, Resistor_SMD:R_0603_1608Metric, symbol Device:R
- added R530: 10k PWM pulldown, Resistor_SMD:R_0603_1608Metric, symbol Device:R
- added SW50, SW51: SWT0210-045026GSA, symbol Switch:SW_Push
- added U50: STM32F401RET6TR, Package_QFP:LQFP-64_10x10mm_P0.5mm, symbol MCU_ST_STM32F4:STM32F401RETx
- U10, U14: symbol Interface_CAN_LIN:MCP2515-xST -> Lab4_Logic:MCP2515_TSSOP20
Connections:
- net +3V3: now also C500.1, C501.1, C502.1, C503.1, C504.1, C505.1, FB50.1, J500.1 (Pin_1), J501.1 (Pin_1), R501.1, R502.1, U50.1 (VBAT), U50.19 (VDD), U50.32 (VDD), U50.48 (VDD), U50.64 (VDD)
- net F_CS_A: now also U50.58 (PB6)
- net F_CS_B: now also U50.38 (PC7)
- net F_INT_A: now also U50.43 (PA10)
- net F_INT_B: now also U50.57 (PB5)
- net F_MISO: now also U50.22 (PA6)
- net F_MOSI: now also U50.23 (PA7)
- net F_SCK: now also U50.21 (PA5)
- net GND: now also C500.2, C501.2, C502.2, C503.2, C504.2, C505.2, C506.2, C507.2, C508.2, C509.2, C510.2, D510.1 (K), D511.1 (K), D512.1 (K), D513.1 (K), J501.3 (Pin_3), J501.6 (Pin_6), J502.3 (Pin_3), J503.1 (Pin_1), J503.2 (Pin_2), J504.1 (Pin_1), J504.2 (Pin_2), J505.1 (Pin_1), J505.2 (Pin_2), R500.2, R530.2, SW50.2, SW51.2, U50.12 (VSSA), U50.18 (VSS), U50.31 (VSS), U50.47 (VSS), U50.63 (VSS)
- net SERVO_ADC: now also J504.8 (Pin_8), U50.16 (PA2)
- new net F_BOOT0: J500.2 (Pin_2), R500.1, U50.60 (BOOT0)
- new net F_DEG_A_LED: J503.7 (Pin_7), R512.1, U50.26 (PB0)
- new net F_DEG_A_LED_ANODE: D512.2 (A), R512.2
- new net F_DEG_B_LED: J503.8 (Pin_8), R513.1, U50.27 (PB1)
- new net F_DEG_B_LED_ANODE: D513.2 (A), R513.2
- new net F_DIR_A_MARKER: J505.4 (Pin_4), U50.29 (PB10)
- new net F_ERROR_LED: J503.13 (Pin_13), J504.4 (Pin_4), R511.1, U50.8 (PC0)
- new net F_ERROR_LED_ANODE: D511.2 (A), R511.2
- new net F_FRONT_LEFT_LED: J503.10 (Pin_10), U50.20 (PA4)
- new net F_FRONT_RIGHT_LED: J503.11 (Pin_11), U50.61 (PB8)
- new net F_PID_MARKER: J504.7 (Pin_7), U50.40 (PC9)
- new net F_PWM_SET_MARKER: J505.3 (Pin_3), U50.62 (PB9)
- new net F_RELAY_TX_MARKER: J503.12 (Pin_12), U50.37 (PC6)
- new net F_RESET_N: C509.1, J501.5 (Pin_5), R501.2, SW50.1, U50.7 (NRST)
- new net F_RX_A_MARKER: J503.3 (Pin_3), U50.10 (PC2)
- new net F_RX_B_MARKER: J503.4 (Pin_4), U50.11 (PC3)
- new net F_SELFTEST_BUTTON: C510.1, J504.3 (Pin_3), R502.2, SW51.1, U50.2 (PC13)
- new net F_SERVO_PWM: J503.9 (Pin_9), R530.1, U50.42 (PA9)
- new net F_STATUS_LED: R510.1, U50.50 (PA15)
- new net F_STATUS_LED_ANODE: D510.2 (A), R510.2
- new net F_STEER_TASK_MARKER: J504.6 (Pin_6), U50.9 (PC1)
- new net F_SWCLK: J501.2 (Pin_2), U50.49 (PA14)
- new net F_SWDIO: J501.4 (Pin_4), U50.46 (PA13)
- new net F_TASK_PROBE: J504.5 (Pin_5), U50.39 (PC8)
- new net F_TX_A_MARKER: J503.5 (Pin_5), U50.14 (PA0)
- new net F_TX_B_MARKER: J503.6 (Pin_6), U50.15 (PA1)
- new net F_UART_CONSOLE_RX: J502.2 (Pin_2), U50.45 (PA12)
- new net F_UART_CONSOLE_TX: J502.1 (Pin_1), U50.44 (PA11)
- new net F_VCAP1: C506.1, U50.30 (VCAP1)
- new net F_VDDA: C507.1, C508.1, FB50.2, U50.13 (VREF+)
- no-connect marks 12 -> 32
Other:
- note added: "LAB3 header follows handout p17 top-to-bottom. Two GND pins first. SRV/PWM_OUT probe actual actuator PWM; timing markers remain separate. Physical header position / accessibility will be checked during PCB layout."
- note added: "STM32F401RET6 - independent HSI/PLL, no ST-LINK clock dependency"
- note added: "SWD: pin1 VTref senses target voltage; do not feed a second 3.3V supply. UART header is TX/RX/GND, not RS-232. NRST pulls low to reset. BOOT0 low boots flash; fit recovery shunt only for bootloader recovery."
- note added: "Servo connector not assigned yet: verify plug order/contact rating. Power is SERVO_PLUS after the shunt; signal F_SERVO_PWM; return GND. Front lamps: PA4 / PB8, output drivers and connectors still pending."
- note added: "Shared rails and CAN backbone connect through the root sheet. SPI, clocks and reset stay within each zone."
- note added: "TEST: active low on PC13, 10k/100n = 1ms release RC. Firmware must debounce and meet the 10ms local-fault deadline. Reset and self-test are separate buttons."
- note added: "VCAP1 is the INTERNAL regulator output. Only its local capacitor connects here. Keep every 100n beside its VDD pin; keep the VCAP loop short. DS10086 Fig.2 / Fig.18."
- note removed: "HOST INTERFACE (to be integrated with the bare MCU / Pi header) SPI1: PA5=SCK, PA6=MISO, PA7=MOSI; PB6=CS_A; PA10=INT_A; PC7=CS_B; PB5=INT_B. These named nets are LOCAL to this zone. All +3V3 / +5V / GND / CAN backbone nets need hierarchy ports before full-board integration."
- title: Front zone - CAN and servo current sensing -> Front zone - integrated logic and interfaces

Commit message: Update Lab 4 circuits, assembly BOMs and measured PCB placement
Parts:
- added J550: FRONT LEFT lamp, Connector_PinHeader_2.54mm:PinHeader_1x02_P2.54mm_Vertical, symbol Connector_Generic:Conn_01x02
- added J551: FRONT RIGHT lamp, Connector_PinHeader_2.54mm:PinHeader_1x02_P2.54mm_Vertical, symbol Connector_Generic:Conn_01x02
- added J90: Servo: GND / 6.6V / PWM, Connector_Hirose:Hirose_DF63M-3P-3.96DSA_1x03_P3.96mm_Vertical, symbol Connector_Generic:Conn_01x03
- added Q550, Q551: MMBT3904, Package_TO_SOT_SMD:SOT-23, symbol Transistor_BJT:MMBT3904
- added R540: 100R, Resistor_SMD:R_0603_1608Metric, symbol Device:R
- added R550, R551: 2.2k, Resistor_SMD:R_0603_1608Metric, symbol Device:R
- added R560, R561: 100k, Resistor_SMD:R_0603_1608Metric, symbol Device:R
- added R570, R571: 220R, Resistor_SMD:R_0603_1608Metric, symbol Device:R
- C100, C101, C140, C141: value Cload TBD -> 18p C0G 50V; Design status (none) -> CL=12pF; equal 18pF caps assume 3pF effective stray; tune a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; MPN (none) -> GRM1885C1H180JA01D
- U11, U15: value SN65HVD231MDREP -> SN65HVD231DR; Design status Course Oct 16 substitution; verify exact supplied ordering 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 -> TI verified SOIC-8 order code; confirm course-stock equival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; MPN SN65HVD231MDREP -> SN65HVD231DR
Connections:
- net F_FRONT_LEFT_LED: now also R550.1
- net F_FRONT_RIGHT_LED: now also R551.1
- net F_SERVO_PWM: now also R540.1
- net GND: now also J90.1 (Pin_1), Q550.2 (E), Q551.2 (E), R560.2, R561.2
- net SERVO_VPLUS: now also J90.2 (Pin_2)
- new net +5V: R570.1, R571.1
- new net F_FRONT_LEFT_LED_BASE: Q550.1 (B), R550.2, R560.1
- new net F_FRONT_LEFT_LED_PLUS: J550.1 (Pin_1), R570.2
- new net F_FRONT_LEFT_LED_SINK: J550.2 (Pin_2), Q550.3 (C)
- new net F_FRONT_RIGHT_LED_BASE: Q551.1 (B), R551.2, R561.1
- new net F_FRONT_RIGHT_LED_PLUS: J551.1 (Pin_1), R571.2
- new net F_FRONT_RIGHT_LED_SINK: J551.2 (Pin_2), Q551.3 (C)
- new net SERVO_PWM_OUT: J90.3 (Pin_3), R540.2
Other:
- note added: "SERVO AND VEHICLE LAMP OUTPUTS"
- note added: "Servo and lamp circuits are below. Connector cable adapters still need physical verification."
- note added: "Servo supply passes through R1. PWM uses PA9 and retains its reset pulldown. J90 uses a new rated 3.96mm connector, not the existing servo plug. Adapter must preserve GND / supply / signal; confirm the servo accepts 3.3V PWM."
- note removed: "Servo connector not assigned yet: verify plug order/contact rating. Power is SERVO_PLUS after the shunt; signal F_SERVO_PWM; return GND. Front lamps: PA4 / PB8, output drivers and connectors still pending."

Commit message: Prepare Lab 4 review package and align course assembly plan
Parts:
- C1, C102, C103, C104, C142, C143, C144, C2: Design status (none) -> Preliminary; verify before fabrication; MPN (none) -> KGM15AR71C104KT
- J1, J11, J15, JP10, JP14, R102, R142, U1, U10, U14: Design status (none) -> Preliminary; verify before fabrication
- Q550, Q551: MPN MMBT3904 -> MMBT3904-7-F
- R1: footprint Resistor_SMD:R_2512_6332Metric -> Lab4_Power:Vishay_WSL2512_7m_to_500m; Design status (none) -> Vishay 30100 p2 land pattern; 10mOhm 1W 1%; 0.16W at 4A; Ke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; MPN (none) -> WSL2512R0100FEA
- R100, R101, R140, R141: Design status (none) -> Preliminary; verify before fabrication; MPN (none) -> CRCW060310K0FKEA
- R2: Design status (none) -> Preliminary; verify before fabrication; MPN (none) -> RC0603FR-074K7L
- SW50, SW51: Design status Electrical circuit placed; exact GCT footprint drawing stil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 -> GCT drawing located (25-Apr-2025); contact-pair/pad geometr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
- U11, U15: Design status TI verified SOIC-8 order code; confirm course-stock equival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 -> Exact MPN appears in course v3 stock list; TI SOIC-8 pinout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

Commit message: Add verified GCT switch footprints and refresh Lab 4 checks
Parts:
- SW50, SW51: footprint (none) -> Lab4_Switches:GCT_SWT0210_4.5x4.5mm; Design status GCT drawing located (25-Apr-2025); contact-pair/pad geometr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 -> GCT A1 drawing verified: physical terminals 1/2 -> logical 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

Commit message: Select approved LiPo pair and add battery voltage monitor
Parts:
- added C580: 100n, Capacitor_SMD:C_0603_1608Metric, symbol Device:C
- added R580: 100k 0.1%, Resistor_SMD:R_0603_1608Metric, symbol Device:R
- added R581: 10k 0.1%, Resistor_SMD:R_0603_1608Metric, symbol Device:R
Connections:
- net GND: now also C580.2, R581.2
- net BATTERY_ADC: now reaches U50.17 (PA3)
- net BATTERY_ADC: now also C580.1, R580.2, R581.1
- new net VBAT_PROTECTED: R580.1
- no-connect marks 32 -> 31
Other:
- note added: "3S LiPo BATTERY MONITOR: protected pack rail / 11 -> PA3 ADC1_IN3. 12.6V full -> 1.145V nominal ADC; 15V ceiling -> 1.364V. Use calibrated VDDA, 480-cycle sample at <=21MHz; allow >=10ms filter settling. No internal pullup/pulldown. Enable BOR; do not treat the MCU VBAT backup pin as pack input. Firmware must inhibit drive at startup, stale/invalid samples and low battery. This is a pack-voltage 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"
